File: dual-ipex-csi-interposer.kicad_pcb (KiCad board)
At the start: 4 copper layers, 26.5 x 64.3 mm, 29 parts, among them J1 WE_68715014522, J2 MSAK24025P30, J3 MSAK24025P30

Commit message: Edit README
Parts:
- C1, C2: footprint antmicro-dual-ipex-csi-interposer-footprints:0402-cap -> dual-ipex-csi-interposer-footprints:0402-cap
- J1: footprint antmicro-dual-ipex-csi-interposer-footprints:WE_68715014522 -> dual-ipex-csi-interposer-footprints:WE_68715014522
- J2, J3: footprint antmicro-dual-ipex-csi-interposer-footprints:MSAK24025P30 -> dual-ipex-csi-interposer-footprints:MSAK24025P30
- MP1, MP2, MP3, MP4: footprint antmicro-dual-ipex-csi-interposer-footprints:mounting-hole-2.2mm -> dual-ipex-csi-interposer-footprints:mounting-hole-2.2mm
- N1: footprint antmicro-dual-ipex-csi-interposer-footprints:oshw-logo -> dual-ipex-csi-interposer-footprints:oshw-logo
- N2: footprint antmicro-dual-ipex-csi-interposer-footprints:antmicro-logo_scaled_12mm -> dual-ipex-csi-interposer-footprints:antmicro-logo_scaled_12mm
- R1, R2, R3, R4, R5, R6, R7, R8: footprint antmicro-dual-ipex-csi-interposer-footprints:0402-res -> dual-ipex-csi-interposer-footprints:0402-res
- TP1, TP10, TP2, TP3, TP4, TP5, TP6, TP7, TP8, TP9: footprint antmicro-dual-ipex-csi-interposer-footprints:Testpoint_smd_1mm -> dual-ipex-csi-interposer-footprints:Testpoint_smd_1mm
