File: dual-ipex-csi-interposer.kicad_sch (KiCad schematic)
At the start: 29 parts, among them J1 WE_68715014522, J2 MSAK24025P30, J3 MSAK24025P30

Commit message: Edit README
Parts:
- C1, C2: footprint antmicro-dual-ipex-csi-interposer-footprints:0402-cap -> dual-ipex-csi-interposer-footprints:0402-cap; symbol antmicro-dual-ipex-csi-interposer:C_100n_0402 -> dual-ipex-csi-interposer:C_100n_0402
- J1: footprint antmicro-dual-ipex-csi-interposer-footprints:WE_68715014522 -> dual-ipex-csi-interposer-footprints:WE_68715014522; symbol antmicro-dual-ipex-csi-interposer:WE_68715014522 -> dual-ipex-csi-interposer:WE_68715014522
- J2, J3: footprint antmicro-dual-ipex-csi-interposer-footprints:MSAK24025P30 -> dual-ipex-csi-interposer-footprints:MSAK24025P30; symbol antmicro-dual-ipex-csi-interposer:MSAK24025P30 -> dual-ipex-csi-interposer:MSAK24025P30
- MP1, MP2, MP3, MP4: footprint antmicro-dual-ipex-csi-interposer-footprints:mounting-hole-2.2mm -> dual-ipex-csi-interposer-footprints:mounting-hole-2.2mm; symbol antmicro-dual-ipex-csi-interposer:PCB_Mount_Hole_2.2_4.5 -> dual-ipex-csi-interposer:PCB_Mount_Hole_2.2_4.5
- N1: footprint antmicro-dual-ipex-csi-interposer-footprints:oshw-logo -> dual-ipex-csi-interposer-footprints:oshw-logo; symbol antmicro-dual-ipex-csi-interposer:oshw_logo -> dual-ipex-csi-interposer:oshw_logo
- N2: footprint antmicro-dual-ipex-csi-interposer-footprints:antmicro-logo_scaled_12mm -> dual-ipex-csi-interposer-footprints:antmicro-logo_scaled_12mm; symbol antmicro-dual-ipex-csi-interposer:antmicro_logo -> dual-ipex-csi-interposer:antmicro_logo
- R1, R2, R3, R4, R5, R6, R7, R8: footprint antmicro-dual-ipex-csi-interposer-footprints:0402-res -> dual-ipex-csi-interposer-footprints:0402-res; symbol antmicro-dual-ipex-csi-interposer:R_0R_0402 -> dual-ipex-csi-interposer:R_0R_0402
- TP1, TP10, TP2, TP3, TP4, TP5, TP6, TP7, TP8, TP9: footprint antmicro-dual-ipex-csi-interposer-footprints:Testpoint_smd_1mm -> dual-ipex-csi-interposer-footprints:Testpoint_smd_1mm; symbol antmicro-dual-ipex-csi-interposer:TP_SMD1MM -> dual-ipex-csi-interposer:TP_SMD1MM
Other:
- note added: "Dual IPEX-CSI interposer"
- note added: "Host CSI connector"
- note added: "IPEX CSI adapter connectors"
- note removed: "Framos CSI adapter connectors"
- note removed: "Framos CSI interposer"
- note removed: "Jetson nano baseboard CSI connector"
- title: (none) -> Dual IPEX-CSI Interposer
